File: kicad/g&w.sch (KiCad schematic (older format))
At the start: 9 parts

Commit message: xrays are fun
Parts:
- removed J?: Conn_01x16, symbol Connector_Generic:Conn_01x16
- removed LS?: Speaker, symbol Device:Speaker
- added C?: C, symbol Device:C
- added J?: DISPLAY1, symbol Connector_Generic:Conn_2Rows-33Pins
- added J?: Conn_01x05, symbol Connector_Generic:Conn_01x05
- added J?: speaker, symbol Connector_Generic:Conn_01x02
- added Q?: MMBT3904, Package_TO_SOT_SMD:SOT-23, symbol Transistor_BJT:MMBT3904
- added R?: R, symbol Device:R
- added R?: 0R, symbol Device:R
- J?: value Conn_01x04 -> DISPLAY2
- J?: value Conn_01x02 -> Battery
Connections:
- net labels added: GND, GNDusb, Vusb
- wire segments 0 -> 18
Other:
- moved on the sheet: J?, U?
Changed lines of the file:
@@
 EELAYER 30 0
 EELAYER END
-$Descr A4 11693 8268
+$Descr A3 16535 11693
 encoding utf-8
 Sheet 1 1
@@
 L Battery_Management:BQ24072RGT U?
 U 1 1 5FC1AF8A
-P 5550 3250
-F 0 "U?" H 5550 4031 50  0000 C CNN
-F 1 "BQ24072RGT" H 5550 3940 50  0000 C CNN
-F 2 "Package_DFN_QFN:VQFN-16-1EP_3x3mm_P0.5mm_EP1.6x1.6mm" H 5850 2700 50  0001 L CNN
-F 3 "http://www.ti.com/lit/ds/symlink/bq24072.pdf" H 5850 3450 50  0001 C CNN
-	1    5550 3250
+P 4650 650
+F 0 "U?" H 4650 1431 50  0000 C CNN
+F 1 "BQ24072RGT" H 4650 1340 50  0000 C CNN
+F 2 "Package_DFN_QFN:VQFN-16-1EP_3x3mm_P0.5mm_EP1.6x1.6mm" H 4950 100 50  0001 L CNN
+F 3 "http://www.ti.com/lit/ds/symlink/bq24072.pdf" H 4950 850 50  0001 C CNN
+	1    4650 650
 	1    0    0    -1
 $EndComp
@@
 L MCU_ST_STM32H7:STM32H743VITx U?
 U 1 1 5FC1F2E4
-P 3750 3550
-F 0 "U?" H 3750 661 50  0000 C CNN
-F 1 "STM32H7B0VGT6" H 3750 570 50  0000 C CNN
-F 2 "Package_QFP:LQFP-100_14x14mm_P0.5mm" H 3050 950 50  0001 R CNN
-F 3 "http://www.st.com/st-web-ui/static/active/en/resource/technical/document/datasheet/DM00387108.pdf" H 3750 3550 50  0001 C CNN
-	1    3750 3550
+P 7950 5300
+F 0 "U?" H 8500 8050 50  0000 C CNN
+F 1 "STM32H7B0VGT6" H 8700 7900 50  0000 C CNN
+F 2 "Package_QFP:LQFP-100_14x14mm_P0.5mm" H 7250 2700 50  0001 R CNN
+F 3 "http://www.st.com/st-web-ui/static/active/en/resource/technical/document/datasheet/DM00387108.pdf" H 7950 5300 50  0001 C CNN
+	1    7950 5300
 	1    0    0    -1
 $EndComp
@@
 L Memory_Flash:MX25R3235FM2xx1 U?
 U 1 1 5FC2EF18
-P 6100 5150
-F 0 "U?" H 6644 5196 50  0000 L CNN
-F 1 "MX25L8035" H 6644 5105 50  0000 L CNN
-F 2 "Package_SO:SOP-8_5.28x5.23mm_P1.27mm" H 6100 4550 50  0001 C CNN
-F 3 "http://www.macronix.com/Lists/Datasheet/Attachments/7534/MX25R3235F,%20Wide%20Range,%2032Mb,%20v1.6.pdf" H 6100 5150 50  0001 C CNN
-	1    6100 5150
+P 5200 2550
+F 0 "U?" H 5744 2596 50  0000 L CNN
+F 1 "MX25L8035" H 5744 2505 50  0000 L CNN
+F 2 "Package_SO:SOP-8_5.28x5.23mm_P1.27mm" H 5200 1950 50  0001 C CNN
+F 3 "http://www.macronix.com/Lists/Datasheet/Attachments/7534/MX25R3235F,%20Wide%20Range,%2032Mb,%20v1.6.pdf" H 5200 2550 50  0001 C CNN
+	1    5200 2550
 	1    0    0    -1
 $EndComp
@@
 L Connector_Generic:Conn_01x04 J?
 U 1 1 5FC33040
-P 7500 2600
-F 0 "J?" H 7580 2592 50  0000 L CNN
-F 1 "Conn_01x04" H 7580 2501 50  0000 L CNN
-F 2 "" H 7500 2600 50  0001 C CNN
-F 3 "~" H 7500 2600 50  0001 C CNN
-	1    7500 2600
-	1    0    0    -1
-$EndComp
-$Comp
-L Connector_Generic:Conn_01x16 J?
-U 1 1 5FC339CE
-P 8550 2400
-F 0 "J?" H 8630 2392 50  0000 L CNN
-F 1 "Conn_01x16" H 8630 2301 50  0000 L CNN
-F 2 "" H 8550 2400 50  0001 C CNN
-F 3 "~" H 8550 2400 50  0001 C CNN
-	1    8550 2400
+P 1900 300
+F 0 "J?" H 1980 292 50  0000 L CNN
+F 1 "DISPLAY2" H 1980 201 50  0000 L CNN
+F 2 "" H 1900 300 50  0001 C CNN
+F 3 "~" H 1900 300 50  0001 C CNN
+	1    1900 300
 	1    0    0    -1
 $EndComp
@@
 L Connector_Generic:Conn_01x02 J?
 U 1 1 5FC365D1
-P 8800 3750
-F 0 "J?" H 8880 3742 50  0000 L CNN
-F 1 "Conn_01x02" H 8880 3651 50  0000 L CNN
-F 2 "" H 8800 3750 50  0001 C CNN
-F 3 "~" H 8800 3750 50  0001 C CNN
-	1    8800 3750
+P 3200 1450
+F 0 "J?" H 3280 1442 50  0000 L CNN
+F 1 "Battery" H 3280 1351 50  0000 L CNN
+F 2 "" H 3200 1450 50  0001 C CNN
+F 3 "~" H 3200 1450 50  0001 C CNN
+	1    3200 1450
 	1    0    0    -1
 $EndComp
@@
 L Connector:USB_C_Receptacle J?
 U 1 1 5FC37056
-P 9950 4700
-F 0 "J?" H 10057 5967 50  0000 C CNN
-F 1 "USB_C_Receptacle" H 10057 5876 50  0000 C CNN
-F 2 "" H 10100 4700 50  0001 C CNN
-F 3 "https://www.usb.org/sites/default/files/documents/usb_type-c.zip" H 10100 4700 50  0001 C CNN
-	1    9950 4700
-	1    0    0    -1
-$EndComp
-$Comp
-L Device:Speaker LS?
-U 1 1 5FC3B588
-P 10000 2100
-F 0 "LS?" H 10170 2096 50  0000 L CNN
-F 1 "Speaker" H 10170 2005 50  0000 L CNN
-F 2 "" H 10000 1900 50  0001 C CNN
-F 3 "~" H 9990 2050 50  0001 C CNN
-	1    10000 2100
+P 1050 5250
+F 0 "J?" H 1157 6517 50  0000 C CNN
+F 1 "USB_C_Receptacle" H 1157 6426 50  0000 C CNN
+F 2 "" H 1200 5250 50  0001 C CNN
+F 3 "https://www.usb.org/sites/default/files/documents/usb_type-c.zip" H 1200 5250 50  0001 C CNN
+	1    1050 5250
 	1    0    0    -1
 $EndComp
@@
 	1    0    0    -1
 $EndComp
+$Comp
+L Connector_Generic:Conn_2Rows-33Pins J?
+U 1 1 5FCB3F0B
+P 7350 1450
+F 0 "J?" H 7400 2467 50  0000 C CNN
+F 1 "DISPLAY1" H 7400 2376 50  0000 C CNN
+F 2 "" H 7350 1450 50  0001 C CNN
+F 3 "~" H 7350 1450 50  0001 C CNN
+	1    7350 1450
+	1    0    0    -1
+$EndComp
+$Comp
+L Transistor_BJT:MMBT3904 Q?
+U 1 1 5FCBC3DE
+P 8800 1600
+F 0 "Q?" H 8991 1646 50  0000 L CNN
+F 1 "MMBT3904" H 8991 1555 50  0000 L CNN
+F 2 "Package_TO_SOT_SMD:SOT-23" H 9000 1525 50  0001 L CIN
+F 3 "https://www.onsemi.com/pub/Collateral/2N3903-D.PDF" H 8800 1600 50  0001 L CNN
+	1    8800 1600
+	1    0    0    -1
+$EndComp
+$Comp
+L Connector_Generic:Conn_01x05 J?
+U 1 1 5FCBD370
+P 1850 1050
+F 0 "J?" H 1930 1092 50  0000 L CNN
+F 1 "Conn_01x05" H 1930 1001 50  0000 L CNN
+F 2 "" H 1850 1050 50  0001 C CNN
+F 3 "~" H 1850 1050 50  0001 C CNN
+	1    1850 1050
+	1    0    0    -1
+$EndComp
+$Comp
+L Connector_Generic:Conn_01x02 J?
+U 1 1 5FCE8178
+P 2450 2450
+F 0 "J?" H 2530 2442 50  0000 L CNN
+F 1 "speaker" H 2530 2351 50  0000 L CNN
+F 2 "" H 2450 2450 50  0001 C CNN
+F 3 "~" H 2450 2450 50  0001 C CNN
+	1    2450 2450
+	1    0    0    -1
+$EndComp
+$Comp
+L Device:R R?
+U 1 1 5FCEB32A
+P 1700 2450
+F 0 "R?" H 1770 2496 50  0000 L CNN
+F 1 "R" H 1770 2405 50  0000 L CNN
+F 2 "" V 1630 2450 50  0001 C CNN
+F 3 "~" H 1700 2450 50  0001 C CNN
+	1    1700 2450
+	1    0    0    -1
+$EndComp
+$Comp
+L Device:C C?
+U 1 1 5FCEBDEF
+P 2300 3000
+F 0 "C?" H 2415 3046 50  0000 L CNN
+F 1 "C" H 2415 2955 50  0000 L CNN
+F 2 "" H 2338 2850 50  0001 C CNN
+F 3 "~" H 2300 3000 50  0001 C CNN
+	1    2300 3000
+	1    0    0    -1
+$EndComp
+Text GLabel 2100 4250 2    50   Input ~ 0
+Vusb
+Text GLabel 1100 7000 2    50   Input ~ 0
+GNDusb
+Wire Wire Line
+	1100 7000 1050 7000
+Wire Wire Line
+	750  7000 750  6850
+Wire Wire Line
+	1050 6850 1050 7000
+Connection ~ 1050 7000
+Wire Wire Line
+	1050 7000 750  7000
+Text GLabel 8350 8300 2    50   Input ~ 0
+GND
+Wire Wire Line
+	7650 8100 7650 8300
+Wire Wire Line
+	7650 8300 7750 8300
+Wire Wire Line
+	8150 8100 8150 8300
+Connection ~ 8150 8300
+Wire Wire Line
+	8150 8300 8350 8300
+Wire Wire Line
+	8050 8100 8050 8300
+Connection ~ 8050 8300
+Wire Wire Line
+	8050 8300 8150 8300
+Wire Wire Line
+	7950 8100 7950 8300
+Connection ~ 7950 8300
+Wire Wire Line
+	7950 8300 8050 8300
+Wire Wire Line
+	7850 8100 7850 8300
+Connection ~ 7850 8300
+Wire Wire Line
+	7850 8300 7950 8300
+Wire Wire Line
+	7750 8100 7750 8300
+Connection ~ 7750 8300
+Wire Wire Line
+	7750 8300 7850 8300
+$Comp
+L Device:R R?
+U 1 1 5FD17E5A
+P 1850 4250
+F 0 "R?" V 1643 4250 50  0000 C CNN
+F 1 "0R" V 1734 4250 50  0000 C CNN
+F 2 "" V 1780 4250 50  0001 C CNN
+F 3 "~" H 1850 4250 50  0001 C CNN
+	1    1850 4250
+	0    1    1    0
+$EndComp
+Wire Wire Line
+	1650 4250 1700 4250
+Wire Wire Line
+	2000 4250 2100 4250
 $EndSCHEMATC

Commit message: Retrace Version 1.0 and spreadsheet pin maps started
Parts:
- added C? (x5): C, symbol Device:C
- added JP?: SolderJumper_2_Bridged, symbol Jumper:SolderJumper_2_Bridged
- added R?: 3k0, symbol Device:R
- added R?: 4k7, symbol Device:R
- added R?: 10R, symbol Device:R
- J?: value Conn_01x05 -> SWD PORT
Connections:
- net labels added: RESET, SWCLK, SWDIO, VCC, Vaux1, d11p66-PC9, d13p47-PB11, d15p84-PD3, d17p34-PB0, d19p68-PA9, d21p45-PE15, d23p51-PB12, d25p41-PE11, d27p63-PC6, d29p54-PB15, d3p55-PD8, d5p57-PD10, d7p91-PB5, d9p83-PD2, dp-P
- wire segments 18 -> 67
- no-connect marks 0 -> 19
Other:
- note added: "33\n32\n31\n30\n29\n28\n27\n26\n25\n24\n23\n22\n21\n20\n19\n18"
- note added: "NW/OLD\n01 = 01\n02 = 33\n03 = 02\n04 = 32\n05 = 03\n06 = 31\n07 = 04\n08 = 30\n09 = 05\n10 = 29\n11 = 06\n12 = 28\n13 = 07\n14 = 27\n15 = 08\n16 = 26\n17 = 09\n18 = 25\n19 = 10\n20 = 24\n21 = 11\n22 = 23\n23 = 12\n24 = 22\n25 = 13\n26 = 21\n27 = 14\n28 = 20\n29 = 15\n30 = 19\n31 = 16\n32 = 18\n33 = 17"
- moved on the sheet: J?, Q?, U?

Commit message: image
Parts:
- U?: value MX25L8035 -> MX25U8035F
Connections:
- net labels added: V1v8, V3v3, Vaux1v8, d10p15-PC0, d12p46-PB10, d14p64-PC7, d16p78-PC10, d18p70-PA11, d20p67-PA8, d24p52-PB13, d25p43-PE13, d26p53-PB14, d28p31-PA7, d4p87-PD6, d6p69-PA10, d8p95-PB8
- net labels removed: Vaux1, d25p41-PE11, dp-P
Other:
- note removed: "33\n32\n31\n30\n29\n28\n27\n26\n25\n24\n23\n22\n21\n20\n19\n18"
- moved on the sheet: U?
Changed lines of the file:
@@
 L Memory_Flash:MX25R3235FM2xx1 U?
 U 1 1 5FC2EF18
-P 5200 6750
-F 0 "U?" H 5744 6796 50  0000 L CNN
-F 1 "MX25L8035" H 5744 6705 50  0000 L CNN
-F 2 "Package_SO:SOP-8_5.28x5.23mm_P1.27mm" H 5200 6150 50  0001 C CNN
-F 3 "http://www.macronix.com/Lists/Datasheet/Attachments/7534/MX25R3235F,%20Wide%20Range,%2032Mb,%20v1.6.pdf" H 5200 6750 50  0001 C CNN
-	1    5200 6750
+P 11800 5950
+F 0 "U?" H 12344 5996 50  0000 L CNN
+F 1 "MX25U8035F" H 12344 5905 50  0000 L CNN
+F 2 "Package_SO:SOP-8_5.28x5.23mm_P1.27mm" H 11800 5350 50  0001 C CNN
+F 3 "http://www.macronix.com/Lists/Datasheet/Attachments/7534/MX25R3235F,%20Wide%20Range,%2032Mb,%20v1.6.pdf" H 11800 5950 50  0001 C CNN
+	1    11800 5950
 	1    0    0    -1
 $EndComp
@@
 $EndComp
 Text GLabel 7550 2400 0    50   Input ~ 0
-VCC
+V1v8
 Wire Wire Line
 	7550 2400 7650 2400
@@
 SWDIO
 Text GLabel 5400 8300 0    50   Input ~ 0
-VCC
+V1v8
 Text GLabel 5400 8200 0    50   Input ~ 0
 GND
@@
 Text GLabel 7050 7300 0    50   Input ~ 0
 d5p57-PD10
-Text Notes 12050 4450 0    63   ~ 0
-33\n32\n31\n30\n29\n28\n27\n26\n25\n24\n23\n22\n21\n20\n19\n18
 Text GLabel 11500 3200 0    50   Input ~ 0
 d7p91-PB5
@@
 Text GLabel 8850 7200 2    50   Input ~ 0
 d11p66-PC9
-Text GLabel 12250 3200 2    50   Input ~ 0
-dp-P
+Text GLabel 12000 3200 2    50   Input ~ 0
+d8p95-PB8
 Text GLabel 11500 3500 0    50   Input ~ 0
 d13p47-PB11
@@
 d23p51-PB12
 Text GLabel 11500 4100 0    50   Input ~ 0
-d25p41-PE11
-Text GLabel 7050 5700 0    50   Input ~ 0
-d25p41-PE11
+d25p43-PE13
+Text GLabel 7050 5900 0    50   Input ~ 0
+d25p43-PE13
 Text GLabel 11500 4200 0    50   Input ~ 0
 d27p63-PC6
@@
 d29p54-PB15
 Text GLabel 11500 4400 0    50   Input ~ 0
-Vaux1
+Vaux1v8
 Text GLabel 11500 4500 0    50   Input ~ 0
 GND
 Text GLabel 10300 5150 0    50   Input ~ 0
-Vaux1
-Text GLabel 12250 2900 2    50   Input ~ 0
-dp-P
-Text GLabel 12250 3000 2    50   Input ~ 0
-dp-P
-Text GLabel 12250 3100 2    50   Input ~ 0
-dp-P
-Text GLabel 12250 3300 2    50   Input ~ 0
-dp-P
-Text GLabel 12250 3400 2    50   Input ~ 0
-dp-P
-Text GLabel 12250 3500 2    50   Input ~ 0
-dp-P
-Text GLabel 12250 3600 2    50   Input ~ 0
-dp-P
-Text GLabel 12250 3700 2    50   Input ~ 0
-dp-P
-Text GLabel 12250 3800 2    50   Input ~ 0
-dp-P
-Text GLabel 12250 3900 2    50   Input ~ 0
-dp-P
-Text GLabel 12250 4000 2    50   Input ~ 0
-dp-P
-Text GLabel 12250 4100 2    50   Input ~ 0
-dp-P
-Text GLabel 12250 4200 2    50   Input ~ 0
-dp-P
-Text GLabel 12250 4300 2    50   Input ~ 0
-dp-P
-Text GLabel 12250 4400 2    50   Input ~ 0
-dp-P
+Vaux1v8
+Text GLabel 12000 3000 2    50   Input ~ 0
+d4p87-PD6
+Text GLabel 12000 3100 2    50   Input ~ 0
+d6p69-PA10
+Text GLabel 12000 3300 2    50   Input ~ 0
+d10p15-PC0
+Text GLabel 12000 3400 2    50   Input ~ 0
+d12p46-PB10
+Text GLabel 12000 3500 2    50   Input ~ 0
+d14p64-PC7
+Text GLabel 12000 3600 2    50   Input ~ 0
+d16p78-PC10
+Text GLabel 12000 3700 2    50   Input ~ 0
+d18p70-PA11
+Text GLabel 12000 3800 2    50   Input ~ 0
+d20p67-PA8
+Text GLabel 12000 4000 2    50   Input ~ 0
+d24p52-PB13
+Text GLabel 12000 4100 2    50   Input ~ 0
+d26p53-PB14
+Text GLabel 12000 4200 2    50   Input ~ 0
+d28p31-PA7
+Text GLabel 12000 2900 2    50   Input ~ 0
+GND
+Text GLabel 12000 3900 2    50   Input ~ 0
+GND
+Text GLabel 12000 4300 2    50   Input ~ 0
+GND
+Text GLabel 12000 4400 2    50   Input ~ 0
+V3v3
+Text GLabel 10200 4950 2    50   Input ~ 0
+V3v3
+Text GLabel 8850 5400 2    50   Input ~ 0
+d8p95-PB8
+Text GLabel 7050 6900 0    50   Input ~ 0
+d4p87-PD6
+Text GLabel 8850 3900 2    50   Input ~ 0
+d6p69-PA10
+Text GLabel 8850 6300 2    50   Input ~ 0
+d10p15-PC0
+Text GLabel 8850 5600 2    50   Input ~ 0
+d12p46-PB10
+Text GLabel 8850 7000 2    50   Input ~ 0
+d14p64-PC7
+Text GLabel 8850 7300 2    50   Input ~ 0
+d16p78-PC10
+Text GLabel 8850 4000 2    50   Input ~ 0
+d18p70-PA11
+Text GLabel 8850 3700 2    50   Input ~ 0
+d20p67-PA8
+Text GLabel 8850 5900 2    50   Input ~ 0
+d24p52-PB13
+Text GLabel 8850 6000 2    50   Input ~ 0
+d26p53-PB14
+Text GLabel 8850 3600 2    50   Input ~ 0
+d28p31-PA7
 $EndSCHEMATC

Commit message: schematic progress
Parts:
- added B1: D-LEFT, symbol Switch:SW_Push
- added B10: POWER, symbol Switch:SW_Push
- added B2: D-DOWN, symbol Switch:SW_Push
- added B3: D-RIGHT, symbol Switch:SW_Push
- added B4: D-UP, symbol Switch:SW_Push
- added B5: ACTION-B, symbol Switch:SW_Push
- added B6: ACTION-A, symbol Switch:SW_Push
- added B7: MENU-SET, symbol Switch:SW_Push
- added B8: MENU-TIME, symbol Switch:SW_Push
- added B9: MENU-GAME, symbol Switch:SW_Push
- added C? (x4): C, symbol Device:C
- added IC4: pmic, symbol gnw_library:pmic
- added JP? (x3): SolderJumper_2_Bridged, symbol Jumper:SolderJumper_2_Bridged
- added JP? (x14): SolderJumper_2_Open, symbol Jumper:SolderJumper_2_Open
- added L?: L, symbol Device:L
- added Q2, Q3: PMBT3904, Package_TO_SOT_SMD:SOT-23, symbol Transistor_BJT:MMBT3904
- added Q4: SSM6J412TU, symbol gnw_library:SSM6J412TU
- added R? (x2): 3k0, symbol Device:R
- added R? (x2): 4k7, symbol Device:R
- added R? (x2): 10R, symbol Device:R
- added R? (x3): 0R, symbol Device:R
- added R? (x12): R, symbol Device:R
- added TP? (x9): TestPoint, symbol Connector:TestPoint
- Q1: renamed from Q?; value MMBT3904 -> PMBT3904
- gave numbers to parts that had none: 8
Connections:
- net labels added: V3v7, b10p22-PA0, b1p58-PD11, b2p61-PD14, b3p62-PD15, b4p81-PD0, b5p86-PD5, b6p56-PD9, b7p7-PC13, b8p33-PC5, b9p16-PC1, bq4p38-PE8, bq7p24-PA2, bq9p37-PE7, f1p41-PE11, f2p59-PD12, f3p1-PE2, f5p35-PB1, f6p36-PB2, f7p23-PA1, kph-p82-PD1, q1b-p30-PA6, q1e-p17-PC2, q2b-p29-PA5, q2e-p18-PC3, q3b-p28-PA4, q3e-p25-PA3
- net labels removed: GNDusb
- wire segments 67 -> 323
- no-connect marks 19 -> 35
Other:
- note removed: "NW/OLD\n01 = 01\n02 = 33\n03 = 02\n04 = 32\n05 = 03\n06 = 31\n07 = 04\n08 = 30\n09 = 05\n10 = 29\n11 = 06\n12 = 28\n13 = 07\n14 = 27\n15 = 08\n16 = 26\n17 = 09\n18 = 25\n19 = 10\n20 = 24\n21 = 11\n22 = 23\n23 = 12\n24 = 22\n25 = 13\n26 = 21\n27 = 14\n28 = 20\n29 = 15\n30 = 19\n31 = 16\n32 = 18\n33 = 17"
- moved on the sheet: C?, IC2, IC5, J1, J2, J3, J4, J?, Q1, R?, UC1, Y?

Commit message: Version 1.12
Parts:
- removed C? (x2): C, symbol Device:C
- removed JP? (x4): SolderJumper_2_Bridged, symbol Jumper:SolderJumper_2_Bridged
- removed JP? (x14): SolderJumper_2_Open, symbol Jumper:SolderJumper_2_Open
- added C? (x10): C, symbol Device:C
- added IC1: audio, symbol gnw_library:audio
- added JP? (x8): jmp-0805, symbol gnw_library:jmp-0805
- added JP? (x24): JMP-0402-OPEN, symbol gnw_library:JMP-0402-OPEN
- added JP? (x5): JMP-0402-CLOSED, symbol gnw_library:JMP-0402-CLOSED
- added R? (x6): R, symbol Device:R
- added TP? (x5): TestPoint, symbol Connector:TestPoint
- R?: value 0R -> R
Connections:
- net labels added: BAT-MESS-p32-PC4, VBAT, aud-b3-p2-PE3, aud-c1-p3-PE4, aud-d1-p5-PE6, aud-d3-p4-PE5, p20-VREF, p21-VDDa, p27-VDD
- net labels removed: VCC
- wire segments 323 -> 436
Other:
- note added: "REGULATOR TODO"
- moved on the sheet: C?, IC5, J1, J6, J?, R?, Y?

Commit message: Version 1.13/designators for R/C's and in-circuit R-meas-vals/kicad0v2
Parts:
- removed C? (x2): C, symbol Device:C
- removed J6: USB_C_Receptacle, symbol Connector:USB_C_Receptacle
- removed JP?: jmp-0805, symbol gnw_library:jmp-0805
- added C1, C2: 100n, Capacitor_SMD:C_0402_1005Metric, symbol Device:C
- added C22: 1u, symbol Device:C
- added C23, C26: 10u, symbol Device:C
- added C3, C31: 1u, Capacitor_SMD:C_0603_1608Metric, symbol Device:C
- added C7: 100n, symbol Device:C
- added IC3: vreg, symbol gnw_library:vreg
- added J6: USB-C, symbol gnw_library:USB-C
- added JP54, JP55, JP58, JP89: JMP-0603-OPEN, symbol gnw_library:JMP-0603-OPEN
- added JP56: JMP-0603-CLOSED, symbol gnw_library:JMP-0603-CLOSED
- added JP57, JP69, JP82, JP85: JMP-0402-CLOSED, symbol gnw_library:JMP-0402-CLOSED
- added JP59, JP60, JP61, JP62, JP63, JP64, JP65, JP66, JP81, JP90: JMP-0402-OPEN, symbol gnw_library:JMP-0402-OPEN
- added R12: 100K, symbol Device:R
- added R9: 100k, symbol Device:R
- added TP51, TP52, TP53, TP54, TP55, TP69: TestPoint, symbol Connector:TestPoint
- C10, C9: renamed from C?; value C -> 22p
- C12, C13, C15, C19, C20, C25: renamed from C?; value C -> 100n
- C14, C16, C18, C33, C6: renamed from C?; value C -> 1u
- C21: renamed from C?; value C -> 10u
- C32: renamed from C?; value C -> 10u; footprint (none) -> Capacitor_SMD:C_0805_2012Metric
- C34: renamed from C?; value C -> 10n
- R1, R2, R4: renamed from R?; value R -> 10M; footprint (none) -> Resistor_SMD:R_0201_0603Metric
- R10: renamed from R?; value R -> 22K
- R11, R15, R16: renamed from R?; value R -> 100K
- R13, R14: renamed from R?; value R -> 2K2
- R17: renamed from R?; value R -> 7K5; footprint (none) -> Resistor_SMD:R_0402_1005Metric
- R18: renamed from R?; value R -> 22K; footprint (none) -> Resistor_SMD:R_0402_1005Metric
- R19: renamed from R?; value R -> 75K; footprint (none) -> Resistor_SMD:R_0402_1005Metric
- R20: renamed from R?; value R -> 3K; footprint (none) -> Resistor_SMD:R_0402_1005Metric
- R22, R25, R28: renamed from R?; value 4k7 -> 4K7
- R23, R24, R27: renamed from R?; value 3k0 -> 3K0
- R3: renamed from R?; value R -> 10K; footprint (none) -> Resistor_SMD:R_0201_0603Metric
- R30: renamed from R?; value R -> 0R; footprint (none) -> Resistor_SMD:R_0603_1608Metric
- R31: renamed from R?; value R -> 0R; footprint (none) -> Resistor_SMD:R_0402_1005Metric
- R32, R33: renamed from R?; value 0R -> 5K2; footprint (none) -> Resistor_SMD:R_0402_1005Metric
- R34: renamed from R?; footprint (none) -> Resistor_SMD:R_0603_1608Metric
- R35: renamed from R?; value R -> 10K
- R5, R6: renamed from R?; value R -> UNKNOWN; footprint (none) -> Resistor_SMD:R_0402_1005Metric
- R8: renamed from R?; value R -> 100k
- Y1: renamed from Y?; value Crystal -> H01717
- gave numbers to parts that had none: 55
Connections:
- net GND: now also C1.2, C2.2, C22.2, C23.2, C26.2, C3.2, C31.2, C7.2, IC3.2 (GND), IC3.5 (TPAD), JP54.1, JP55.2, JP58.1, JP59.1, JP60.2, JP61.2, JP62.2, JP63.2, JP64.2, JP65.2, JP66.2, JP81.2, JP89.1, JP90.1, R12.1, TP53.1
- net V1v8: now also UC1.100 (VDD), UC1.50 (VDD), UC1.75 (VDD), C26.1, JP82.2; no longer IC4.B3 (VOUT), L1.2
- net V3v3: now also JP57.2, JP58.2, JP59.2, TP55.1
- net V3v7: now also C1.1, C2.1, C3.1, IC3.4 (VIN)
- net VBAT: now also JP81.1
- net Vaux1v8: now also C22.1, JP85.2, JP89.2, JP90.2, R9.2, TP69.1; no longer Q4.5, Q4.6
- net Vusb: now also IC5.13 (IN), C31.1, JP56.2, TP54.1
- net d23p51-PB12: now also R9.1
- net d24p52-PB13: now also JP63.1
- net d25p43-PE13: now also JP64.1
- net d26p53-PB14: now also JP62.1, JP65.1, JP69.2; no longer UC1.53 (PB14)
- net d27p63-PC6: now also JP66.1
- net d28p31-PA7: now also JP61.1
- net d29p54-PB15: now also JP60.1
- net d3p55-PD8: now also C7.1
- net p27-VDD: now also JP54.2
- net lreg3p85-PD4: now reaches UC1.85 (PD4)
- net lreg3p85-PD4: now also IC3.3 (EN), JP55.1, R12.2, TP51.1
- net at R34.2: now also J6.A1 (GND), J6.A12 (GND), J6.B1 (GND), J6.B12 (GND), J6.S1 (SHIELD)
- net at R31.2: now also J6.A4 (VBUS), J6.A9 (VBUS), J6.B4 (VBUS), J6.B9 (VBUS), TP52.1
- net at R33.2: now also J6.A5 (CC1)
- net at R32.1: now also J6.B5 (CC2)
- net at R31.1: now also JP56.1
- new net: JP69.1, UC1.53 (PB14)
- new net: IC4.B3 (VOUT), JP82.1, L1.2
- new net: C23.1, IC3.1 (VOUT), JP57.1
- new net: JP85.1, Q4.5, Q4.6
Other:
- note added: "DISPLAY-CONN-SIDE"
- note added: "uC-SIDE"
- note removed: "REGULATOR TODO"
- moved on the sheet: C18, C6, IC1, J1, J2, R1, R2, R3, R31, R32, R33, R34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
