File: kicad/g&w.sch (KiCad schematic (older format))
At the start: 161 parts, among them IC1 audio, IC2 MX25U8035F, IC3 vreg, IC4 pmic, IC5 BQ24072RGT, J1 speaker, J2 SWD PORT, J3 DISPLAY1, J4 DISPLAY2, J5 Battery, J6 USB-C, Q1 PMBT3904, Q2 PMBT3904, Q3 PMBT3904, Q4 SSM6J412TU, Y1 H01717

Commit message: 4 footprints left to create b4 layout begins
Parts:
- added C11, C17, C30, C4, C5, C8: 100n, Capacitor_SMD:C_0201_0603Metric, symbol Device:C
- added C24, C27: 1u, Capacitor_SMD:C_0402_1005Metric, symbol Device:C
- added C28: 10u, Capacitor_SMD:C_0603_1608Metric, symbol Device:C
- added C29: 22u, Capacitor_SMD:C_0805_2012Metric, symbol Device:C
- added TP71, TP72, TP73, TP74, TP75, TP76, TP77, TP78, TP79, TP80: TestPoint, TestPoint:TestPoint_Pad_D1.0mm, symbol Connector:TestPoint
- B1, B2, B3, B4, B7, B8, B9: footprint (none) -> gnw:Button_Carbon-Contact_Round_5.00mm
- B5, B6: footprint (none) -> gnw:Button_Carbon-Contact_Round_6.5mm
- C1, C2: footprint Capacitor_SMD:C_0402_1005Metric -> Capacitor_SMD:C_0201_0603Metric
- C10, C12, C13, C15, C19, C20, C25, C34, C7, C9: footprint (none) -> Capacitor_SMD:C_0201_0603Metric
- C14, C16, C18, C22, C33, C6: footprint (none) -> Capacitor_SMD:C_0402_1005Metric
- C21, C23, C26: footprint (none) -> Capacitor_SMD:C_0603_1608Metric
- IC1, IC4: footprint (none) -> Package_BGA:Texas_DSBGA-12_1.36x1.86mm_Layout3x4_P0.5mm
- IC3: footprint (none) -> Package_SON:Texas_X2SON-4_1x1mm_P0.65mm
- J1: footprint (none) -> gnw:Speaker
- J2: footprint (none) -> Connector_PinHeader_1.27mm:PinHeader_1x05_P1.27mm_Vertical
- J5: footprint (none) -> Connector_Molex:Molex_Pico-EZmate_78171-0002_1x02-1MP_P1.20mm_Vertical
- JP100, JP101, JP103, JP104, JP105, JP59, JP60, JP61, JP62, JP63, JP64, JP65, JP66, JP68, JP71, JP74, JP75, JP76, JP78, JP79, JP80, JP81, JP86, JP87, JP90, JP91, JP92, JP93, JP94, JP95, JP96, JP97, JP98, JP99: footprint (none) -> Resistor_SMD:R_0402_1005Metric_Pad0.72x0.64mm_HandSolder
- JP102, JP51, JP52, JP53, JP77, JP83, JP84: footprint (none) -> gnw:JMP-0805-CLOSED
- JP54, JP55, JP58, JP89: footprint (none) -> Resistor_SMD:R_0603_1608Metric_Pad0.98x0.95mm_HandSolder
- JP56: footprint (none) -> gnw:JMP-0603-CLOSED
- JP57, JP67, JP69, JP70, JP72, JP73, JP82, JP85, JP88: footprint (none) -> gnw:JMP-0402-CLOSED
- L1: footprint (none) -> Inductor_SMD:L_1008_2520Metric_Pad1.43x2.20mm_HandSolder
- Q4: footprint (none) -> gnw:Toshiba_UF6_SOT363F
- R10, R11, R12, R13, R14, R15, R16, R21, R22, R23, R24, R25, R26, R27, R28, R29, R35, R8, R9: footprint (none) -> Resistor_SMD:R_0201_0603Metric
- R17, R18, R19, R20, R32, R33, R5, R6: footprint Resistor_SMD:R_0402_1005Metric -> Resistor_SMD:R_0201_0603Metric
- R30: footprint Resistor_SMD:R_0603_1608Metric -> Resistor_SMD:R_0402_1005Metric
- TP51, TP52, TP53, TP54, TP55, TP56, TP57, TP58, TP59, TP60, TP61, TP62, TP63, TP64, TP65, TP66, TP67, TP68, TP69, TP70: footprint (none) -> TestPoint:TestPoint_Pad_D1.0mm
- Y1: footprint (none) -> Crystal:Crystal_SMD_3215-2Pin_3.2x1.5mm
Connections:
- net GND: now also C11.2, C17.2, C24.2, C27.2, C28.2, C29.2, C30.2, C4.2, C5.2, C8.2
- net V1v8: now also C11.1, C17.1, C4.1, C5.1, C8.1
- net V3v7: now also C24.1, C27.1, C28.1, C29.1, C30.1
- net b10p22-PA0: now also TP71.1
- net b1p58-PD11: now also TP72.1
- net b2p61-PD14: now also TP73.1
- net b3p62-PD15: now also TP74.1
- net b4p81-PD0: now also TP75.1
- net b5p86-PD5: now also TP76.1
- net b6p56-PD9: now also TP77.1
- net b7p7-PC13: now also TP78.1
- net b8p33-PC5: now also TP79.1
- net b9p16-PC1: now also TP80.1
- net RESET renamed RESET-p14-NRST
- net SWCLK renamed SWCLK-p76-PA14
- net SWDIO renamed SWDIO-p72-PA13
Other:
- moved on the sheet: C7, R9

Commit message: trace 1v14/Schematic 1v0/layout begins
Parts:
- removed IC5: BQ24072RGT, Package_DFN_QFN:VQFN-16-1EP_3x3mm_P0.5mm_EP1.6x1.6mm, symbol Battery_Management:BQ24072RGT
- added IC5: BQ24072RGT_, Package_DFN_QFN:VQFN-16-1EP_3x3mm_P0.5mm_EP1.6x1.6mm, symbol gnw_library:BQ24072RGT_
- B10: footprint (none) -> gnw:SW_PUSH_1P1T_Horizontal_Nintendo_GnW
- J3: footprint (none) -> gnw:Molex_502078-3310_2Rows-33Pins-1MP_P0.5mm-int0.25mm_Horizontal
- J4: footprint (none) -> gnw:Molex_Easy-On_503480-0400_1x04-1MP_P1.00mm_Horizontal
- J6: footprint (none) -> gnw:USB_C_Receptacle_NintendoG&W
- L1: value L -> UNKNOWN
Connections:
- net GND: now also JP55.1, IC5.14 (TMR), IC5.15 (TD), IC5.17 (VSS), IC5.6 (EN1), IC5.8 (VSS); no longer JP55.2, JP78.2, JP79.2, JP86.2, JP87.1, R1.1, R2.2, R3.1, R4.2
- net V3v7: now also IC1.D2 (VDD), IC5.10 (OUT), IC5.11 (OUT)
- net VBAT: now also IC5.2 (BAT), IC5.3 (BAT)
- net Vusb: now also IC5.13 (VIN)
- net aud-b3-p2-PE3: now also IC1.B3 (SAI-SD-B)
- net aud-c1-p3-PE4: now also IC1.C1 (SAI-FS-A)
- net aud-d1-p5-PE6: now also IC1.D1 (SAI-SD-A)
- net bq4p38-PE8: now also IC5.4 (~CE)
- net bq7p24-PA2: now also IC5.7 (~PGOOD)
- net bq9p37-PE7: now also IC5.9 (~CHG)
- net lreg3p85-PD4: now also JP55.2; no longer JP55.1
- net at JP88.1, TP68.1: now also IC5.1 (TS)
- net at R17.2: now also IC5.12 (ILIM)
- net at R20.1: now also IC5.16 (ISET)
- net at JP71.2, R18.2: now also IC5.5 (EN2)
- net at J1.2 (Pin_2), JP84.2: now also JP86.2; no longer JP86.1
- net at IC1.A1 (SPKR-): now also JP84.1
- net at IC1.A2 (GND): now also IC1.C3 (GND), JP78.1, JP79.1, JP86.1, JP87.1, R1.1, R2.2, R3.1, R4.2
- net at IC1.B1 (?): now also JP79.2, JP80.2
- net at IC1.D3 (SAI-SCK-A): now also JP77.2, JP78.2, R4.1
- net at Q4.1: now also JP85.1, Q4.2, Q4.5, Q4.6
- net BAT-MESS-p32-PC4 renamed BAT-MEAS-p32-PC4
- no-connect marks 35 -> 33
Other:
- note added: "NOTES:\nAll resistors were measured in circuit from both directions. If both readings were within ~20%-30% they were given values. The values were chosen with a bias towards common values. The two battery measurement resistors gave no reading, \nand the 10M's for the audio IC are highly suspect, the others seem fairly reliable. All capacitor values are absolute guesses and were not measured. Also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"
- moved on the sheet: C1, C11, C17, C19, C2, C24, C25, C26, C27, C28, C29, C3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
